Commit message: Updating vision module

File: kortex_move_it_config/gen3_move_it_config/config/7dof/gen3.srdf.xacro (robot description, xacro)
@@ -4,6 +4,5 @@
     A URDF file must exist for this robot as well, where the joints and the links that are referenced are defined
 -->
-<robot name="gen3" xmlns:xacro="http://www.ros.org/wiki/xacro">
-    <xacro:arg name="prefix" default="" />
+<robot name="gen3">
     <!--GROUPS: Representation of a set of joints and links. This can be useful for specifying DOF to plan for, defining arms, end effectors, etc-->
     <!--LINKS: When a link is specified, the parent joint of that link (if it exists) is automatically included-->
@@ -12,64 +11,64 @@
     <!--SUBGROUPS: Groups can also be formed by referencing to already defined group names-->
     <group name="arm">
-        <joint name="$(arg prefix)joint_1" />
-        <joint name="$(arg prefix)joint_2" />
-        <joint name="$(arg prefix)joint_3" />
-        <joint name="$(arg prefix)joint_4" />
-        <joint name="$(arg prefix)joint_5" />
-        <joint name="$(arg prefix)joint_6" />
-        <joint name="$(arg prefix)joint_7" />
-        <joint name="$(arg prefix)end_effector" />
-        <joint name="$(arg prefix)tool_frame_joint" />
+        <joint name="joint_1" />
+        <joint name="joint_2" />
+        <joint name="joint_3" />
+        <joint name="joint_4" />
+        <joint name="joint_5" />
+        <joint name="joint_6" />
+        <joint name="joint_7" />
+        <joint name="end_effector" />
+        <joint name="tool_frame_joint" />
     </group>
     <!--GROUP STATES: Purpose: Define a named state for a particular group, in terms of joint values. This is useful to define states like 'folded arms'-->
     <group_state name="home" group="arm">
-        <joint name="$(arg prefix)joint_1" value="0" />
-        <joint name="$(arg prefix)joint_2" value="0.26" />
-        <joint name="$(arg prefix)joint_3" value="3.14" />
-        <joint name="$(arg prefix)joint_4" value="-2.27" />
-        <joint name="$(arg prefix)joint_5" value="0" />
-        <joint name="$(arg prefix)joint_6" value="0.96" />
-        <joint name="$(arg prefix)joint_7" value="1.57" />
+        <joint name="joint_1" value="0" />
+        <joint name="joint_2" value="0.26" />
+        <joint name="joint_3" value="3.14" />
+        <joint name="joint_4" value="-2.27" />
+        <joint name="joint_5" value="0" />
+        <joint name="joint_6" value="0.96" />
+        <joint name="joint_7" value="1.57" />
     </group_state>
     <group_state name="retract" group="arm">
-        <joint name="$(arg prefix)joint_1" value="0" />
-        <joint name="$(arg prefix)joint_2" value="-0.35" />
-        <joint name="$(arg prefix)joint_3" value="3.14" />
-        <joint name="$(arg prefix)joint_4" value="-2.54" />
-        <joint name="$(arg prefix)joint_5" value="0" />
-        <joint name="$(arg prefix)joint_6" value="-0.87" />
-        <joint name="$(arg prefix)joint_7" value="1.57" />
+        <joint name="joint_1" value="0" />
+        <joint name="joint_2" value="-0.35" />
+        <joint name="joint_3" value="3.14" />
+        <joint name="joint_4" value="-2.54" />
+        <joint name="joint_5" value="0" />
+        <joint name="joint_6" value="-0.87" />
+        <joint name="joint_7" value="1.57" />
     </group_state>
     <group_state name="vertical" group="arm">
-        <joint name="$(arg prefix)joint_1" value="0" />
-        <joint name="$(arg prefix)joint_2" value="0" />
-        <joint name="$(arg prefix)joint_3" value="0" />
-        <joint name="$(arg prefix)joint_4" value="0" />
-        <joint name="$(arg prefix)joint_5" value="0" />
-        <joint name="$(arg prefix)joint_6" value="0" />
-        <joint name="$(arg prefix)joint_7" value="0" />
+        <joint name="joint_1" value="0" />
+        <joint name="joint_2" value="0" />
+        <joint name="joint_3" value="0" />
+        <joint name="joint_4" value="0" />
+        <joint name="joint_5" value="0" />
+        <joint name="joint_6" value="0" />
+        <joint name="joint_7" value="0" />
     </group_state>
     <!--DISABLE COLLISIONS: By default it is assumed that any link of the robot could potentially come into collision with any other link in the robot. This tag disables collision checking between a specified pair of links. -->
-    <disable_collisions link1="$(arg prefix)bracelet_link" link2="$(arg prefix)forearm_link" reason="Never" />
-    <disable_collisions link1="$(arg prefix)bracelet_link" link2="$(arg prefix)spherical_wrist_1_link" reason="Never" />
-    <disable_collisions link1="$(arg prefix)bracelet_link" link2="$(arg prefix)spherical_wrist_2_link" reason="Adjacent" />
-    <disable_collisions link1="$(arg prefix)forearm_link" link2="$(arg prefix)half_arm_1_link" reason="Never" />
-    <disable_collisions link1="$(arg prefix)forearm_link" link2="$(arg prefix)half_arm_2_link" reason="Adjacent" />
-    <disable_collisions link1="$(arg prefix)forearm_link" link2="$(arg prefix)shoulder_link" reason="Never" />
-    <disable_collisions link1="$(arg prefix)forearm_link" link2="$(arg prefix)spherical_wrist_1_link" reason="Adjacent" />
-    <disable_collisions link1="$(arg prefix)forearm_link" link2="$(arg prefix)spherical_wrist_2_link" reason="Never" />
-    <disable_collisions link1="$(arg prefix)forearm_link" link2="$(arg prefix)base_link" reason="Never" />
-    <disable_collisions link1="$(arg prefix)half_arm_1_link" link2="$(arg prefix)half_arm_2_link" reason="Adjacent" />
-    <disable_collisions link1="$(arg prefix)half_arm_1_link" link2="$(arg prefix)shoulder_link" reason="Adjacent" />
-    <disable_collisions link1="$(arg prefix)half_arm_1_link" link2="$(arg prefix)spherical_wrist_1_link" reason="Never" />
-    <disable_collisions link1="$(arg prefix)half_arm_1_link" link2="$(arg prefix)spherical_wrist_2_link" reason="Never" />
-    <disable_collisions link1="$(arg prefix)half_arm_1_link" link2="$(arg prefix)base_link" reason="Never" />
-    <disable_collisions link1="$(arg prefix)half_arm_2_link" link2="$(arg prefix)shoulder_link" reason="Never" />
-    <disable_collisions link1="$(arg prefix)half_arm_2_link" link2="$(arg prefix)spherical_wrist_1_link" reason="Never" />
-    <disable_collisions link1="$(arg prefix)half_arm_2_link" link2="$(arg prefix)spherical_wrist_2_link" reason="Never" />
-    <disable_collisions link1="$(arg prefix)half_arm_2_link" link2="$(arg prefix)base_link" reason="Never" />
-    <disable_collisions link1="$(arg prefix)shoulder_link" link2="$(arg prefix)spherical_wrist_1_link" reason="Never" />
-    <disable_collisions link1="$(arg prefix)shoulder_link" link2="$(arg prefix)spherical_wrist_2_link" reason="Never" />
-    <disable_collisions link1="$(arg prefix)shoulder_link" link2="$(arg prefix)base_link" reason="Adjacent" />
-    <disable_collisions link1="$(arg prefix)spherical_wrist_1_link" link2="$(arg prefix)spherical_wrist_2_link" reason="Adjacent" />
+    <disable_collisions link1="base_link" link2="forearm_link" reason="Never" />
+    <disable_collisions link1="base_link" link2="half_arm_1_link" reason="Never" />
+    <disable_collisions link1="base_link" link2="half_arm_2_link" reason="Never" />
+    <disable_collisions link1="base_link" link2="shoulder_link" reason="Adjacent" />
+    <disable_collisions link1="bracelet_link" link2="forearm_link" reason="Never" />
+    <disable_collisions link1="bracelet_link" link2="spherical_wrist_1_link" reason="Never" />
+    <disable_collisions link1="bracelet_link" link2="spherical_wrist_2_link" reason="Adjacent" />
+    <disable_collisions link1="forearm_link" link2="half_arm_1_link" reason="Never" />
+    <disable_collisions link1="forearm_link" link2="half_arm_2_link" reason="Adjacent" />
+    <disable_collisions link1="forearm_link" link2="shoulder_link" reason="Never" />
+    <disable_collisions link1="forearm_link" link2="spherical_wrist_1_link" reason="Adjacent" />
+    <disable_collisions link1="forearm_link" link2="spherical_wrist_2_link" reason="Never" />
+    <disable_collisions link1="half_arm_1_link" link2="half_arm_2_link" reason="Adjacent" />
+    <disable_collisions link1="half_arm_1_link" link2="shoulder_link" reason="Adjacent" />
+    <disable_collisions link1="half_arm_1_link" link2="spherical_wrist_1_link" reason="Never" />
+    <disable_collisions link1="half_arm_1_link" link2="spherical_wrist_2_link" reason="Never" />
+    <disable_collisions link1="half_arm_2_link" link2="shoulder_link" reason="Never" />
+    <disable_collisions link1="half_arm_2_link" link2="spherical_wrist_1_link" reason="Never" />
+    <disable_collisions link1="half_arm_2_link" link2="spherical_wrist_2_link" reason="Never" />
+    <disable_collisions link1="shoulder_link" link2="spherical_wrist_1_link" reason="Never" />
+    <disable_collisions link1="shoulder_link" link2="spherical_wrist_2_link" reason="Never" />
+    <disable_collisions link1="spherical_wrist_1_link" link2="spherical_wrist_2_link" reason="Adjacent" />
 </robot>
